File: PCB Design/mcu.sch (KiCad schematic (older format))
At the start: 10 parts, among them P14 CONN_01X06, U4 dsPIC33FJ32GS606, X2 10MHz

Commit message: Added initial footprint associations, caps and resistors.
Kicad is giving weird errors for the libraries and BOM generator.
The libraries have to be downloaded manually from github, and
then added.

Signed-off-by: Kolijn Wolfaardt <kolijn.wolfaardt@gmail.com>
Parts:
- C18, C19, C20, C21: footprint (none) -> Capacitors_SMD:C_1206
- P14: footprint (none) -> Pin_Headers:Pin_Header_Straight_1x06
- R13, R14: footprint (none) -> Resistors_SMD:R_1206
- RESET1: footprint (none) -> Buttons_Switches_SMD:SW_SPST_PTS645
- U4: footprint (none) -> TQFP
Changed lines of the file:
@@
 F 0 "U4" H 5200 3650 60  0000 C CNN
 F 1 "dsPIC33FJ32GS606" H 5150 150 60  0000 C CNN
-F 2 "" H 5200 2400 60  0000 C CNN
+F 2 "TQFP" H 5200 2400 60  0001 C CNN
 F 3 "" H 5200 2400 60  0000 C CNN
 	1    5200 2400
@@
 F 0 "P14" H 1600 6750 50  0000 C CNN
 F 1 "CONN_01X06" V 1700 6400 50  0000 C CNN
-F 2 "" H 1600 6400 60  0000 C CNN
+F 2 "Pin_Headers:Pin_Header_Straight_1x06" H 1600 6400 60  0001 C CNN
 F 3 "" H 1600 6400 60  0000 C CNN
 	1    1600 6400
@@
 F 0 "X2" H 3950 6290 50  0000 C CNN
 F 1 "10MHz" H 3980 6090 50  0000 L CNN
-F 2 "" H 3950 6200 60  0000 C CNN
+F 2 "" H 3950 6200 60  0001 C CNN
 F 3 "" H 3950 6200 60  0000 C CNN
 	1    3950 6200
@@
 F 0 "C18" H 4300 6000 50  0000 L CNN
 F 1 "22pF" H 4300 5800 50  0000 L CNN
-F 2 "" H 4288 5750 30  0000 C CNN
+F 2 "Capacitors_SMD:C_1206" H 4288 5750 30  0001 C CNN
 F 3 "" H 4250 5900 60  0000 C CNN
 	1    4250 5900
@@
 F 0 "C19" H 4300 6600 50  0000 L CNN
 F 1 "22pF" H 4300 6400 50  0000 L CNN
-F 2 "" H 4288 6350 30  0000 C CNN
+F 2 "Capacitors_SMD:C_1206" H 4288 6350 30  0001 C CNN
 F 3 "" H 4250 6500 60  0000 C CNN
 	1    4250 6500
@@
 F 0 "C20" H 6150 6500 50  0000 L CNN
 F 1 "10uF" H 6150 6300 50  0000 L CNN
-F 2 "" H 6138 6250 30  0000 C CNN
+F 2 "Capacitors_SMD:C_1206" H 6138 6250 30  0001 C CNN
 F 3 "" H 6100 6400 60  0000 C CNN
 	1    6100 6400
@@
 F 0 "RESET1" H 10200 3100 50  0000 C CNN
 F 1 "DPST" H 10200 3000 50  0000 C CNN
-F 2 "" H 9900 3050 60  0000 C CNN
+F 2 "Buttons_Switches_SMD:SW_SPST_PTS645" H 9900 3050 60  0001 C CNN
 F 3 "" H 9900 3050 60  0000 C CNN
 	1    9900 3050
@@
 F 0 "R13" V 9030 2450 50  0000 C CNN
 F 1 "220" V 8957 2451 50  0000 C CNN
-F 2 "" V 8880 2450 30  0000 C CNN
+F 2 "Resistors_SMD:R_1206" V 8880 2450 30  0001 C CNN
 F 3 "" H 8950 2450 30  0000 C CNN
 	1    8950 2450
@@
 F 0 "R14" V 9780 2100 50  0000 C CNN
 F 1 "4.7k" V 9707 2101 50  0000 C CNN
-F 2 "" V 9630 2100 30  0000 C CNN
+F 2 "Resistors_SMD:R_1206" V 9630 2100 30  0001 C CNN
 F 3 "" H 9700 2100 30  0000 C CNN
 	1    9700 2100
@@
 F 0 "C21" H 9400 2850 50  0000 L CNN
 F 1 "100nF" H 9400 2650 50  0000 L CNN
-F 2 "" H 9388 2600 30  0000 C CNN
+F 2 "Capacitors_SMD:C_1206" H 9388 2600 30  0001 C CNN
 F 3 "" H 9350 2750 60  0000 C CNN
 	1    9350 2750

Commit message: Added diodes to motor driver
Signed-off-by: Kolijn_Laptop <kolijn.wolfaardt@gmail.com>
Parts:
- U4: footprint TQFP -> Housings_QFP:TQFP-64_10x10mm_Pitch0.5mm
Changed lines of the file:
@@
 F 0 "U4" H 5200 3650 60  0000 C CNN
 F 1 "dsPIC33FJ32GS606" H 5150 150 60  0000 C CNN
-F 2 "TQFP" H 5200 2400 60  0001 C CNN
+F 2 "Housings_QFP:TQFP-64_10x10mm_Pitch0.5mm" H 5200 2400 60  0001 C CNN
 F 3 "" H 5200 2400 60  0000 C CNN
 	1    5200 2400
@@
 $EndComp
 $Comp
-L +3V3 #PWR050
+L +3V3 #PWR053
 U 1 1 550F44AC
 P 2400 6150
-F 0 "#PWR050" H 2400 6000 60  0001 C CNN
+F 0 "#PWR053" H 2400 6000 60  0001 C CNN
 F 1 "+3V3" H 2400 6290 60  0000 C CNN
 F 2 "" H 2400 6150 60  0000 C CNN
@@
 $EndComp
 $Comp
-L GND #PWR051
+L GND #PWR054
 U 1 1 550F44B3
 P 2400 6450
-F 0 "#PWR051" H 2400 6200 60  0001 C CNN
+F 0 "#PWR054" H 2400 6200 60  0001 C CNN
 F 1 "GND" H 2400 6300 60  0000 C CNN
 F 2 "" H 2400 6450 60  0000 C CNN
@@
 MCLR_in
 $Comp
-L +3V3 #PWR052
+L +3V3 #PWR055
 U 1 1 550F44C2
 P 2250 3700
-F 0 "#PWR052" H 2250 3550 60  0001 C CNN
+F 0 "#PWR055" H 2250 3550 60  0001 C CNN
 F 1 "+3V3" H 2250 3840 60  0000 C CNN
 F 2 "" H 2250 3700 60  0000 C CNN
@@
 $EndComp
 $Comp
-L GND #PWR053
+L GND #PWR056
 U 1 1 550F44C8
 P 2000 4350
-F 0 "#PWR053" H 2000 4100 60  0001 C CNN
+F 0 "#PWR056" H 2000 4100 60  0001 C CNN
 F 1 "GND" H 2000 4200 60  0000 C CNN
 F 2 "" H 2000 4350 60  0000 C CNN
@@
 $EndComp
 $Comp
-L +3V3 #PWR054
+L +3V3 #PWR057
 U 1 1 550F44D2
 P 2200 2000
-F 0 "#PWR054" H 2200 1850 60  0001 C CNN
+F 0 "#PWR057" H 2200 1850 60  0001 C CNN
 F 1 "+3V3" H 2200 2140 60  0000 C CNN
 F 2 "" H 2200 2000 60  0000 C CNN
@@
 $EndComp
 $Comp
-L GND #PWR055
+L GND #PWR058
 U 1 1 550F44D8
 P 2000 2650
-F 0 "#PWR055" H 2000 2400 60  0001 C CNN
+F 0 "#PWR058" H 2000 2400 60  0001 C CNN
 F 1 "GND" H 2000 2500 60  0000 C CNN
 F 2 "" H 2000 2650 60  0000 C CNN
@@
 $EndComp
 $Comp
-L +3V3 #PWR056
+L +3V3 #PWR059
 U 1 1 550F44E2
 P 8000 3950
-F 0 "#PWR056" H 8000 3800 60  0001 C CNN
+F 0 "#PWR059" H 8000 3800 60  0001 C CNN
 F 1 "+3V3" H 8000 4090 60  0000 C CNN
 F 2 "" H 8000 3950 60  0000 C CNN
@@
 $EndComp
 $Comp
-L GND #PWR057
+L GND #PWR060
 U 1 1 550F44E8
 P 7800 3700
-F 0 "#PWR057" H 7800 3450 60  0001 C CNN
+F 0 "#PWR060" H 7800 3450 60  0001 C CNN
 F 1 "GND" H 7800 3550 60  0000 C CNN
 F 2 "" H 7800 3700 60  0000 C CNN
@@
 $EndComp
 $Comp
-L +3V3 #PWR058
+L +3V3 #PWR061
 U 1 1 550F44F1
 P 7850 1900
-F 0 "#PWR058" H 7850 1750 60  0001 C CNN
+F 0 "#PWR061" H 7850 1750 60  0001 C CNN
 F 1 "+3V3" H 7850 2040 60  0000 C CNN
 F 2 "" H 7850 1900 60  0000 C CNN
@@
 PGC
 $Comp
-L +3V3 #PWR059
+L +3V3 #PWR062
 U 1 1 550F450D
 P 2100 3100
-F 0 "#PWR059" H 2100 2950 60  0001 C CNN
+F 0 "#PWR062" H 2100 2950 60  0001 C CNN
 F 1 "+3V3" H 2100 3240 60  0000 C CNN
 F 2 "" H 2100 3100 60  0000 C CNN
@@
 $EndComp
 $Comp
-L GND #PWR060
+L GND #PWR063
 U 1 1 550F4513
 P 2100 3350
-F 0 "#PWR060" H 2100 3100 60  0001 C CNN
+F 0 "#PWR063" H 2100 3100 60  0001 C CNN
 F 1 "GND" H 2100 3200 60  0000 C CNN
 F 2 "" H 2100 3350 60  0000 C CNN
@@
 $EndComp
 $Comp
-L GND #PWR061
+L GND #PWR064
 U 1 1 550F453B
 P 4550 6600
-F 0 "#PWR061" H 4550 6350 60  0001 C CNN
+F 0 "#PWR064" H 4550 6350 60  0001 C CNN
 F 1 "GND" H 4550 6450 60  0000 C CNN
 F 2 "" H 4550 6600 60  0000 C CNN
@@
 $EndComp
 $Comp
-L GND #PWR062
+L GND #PWR065
 U 1 1 550F4558
 P 6100 6700
-F 0 "#PWR062" H 6100 6450 60  0001 C CNN
+F 0 "#PWR065" H 6100 6450 60  0001 C CNN
 F 1 "GND" H 6100 6550 60  0000 C CNN
 F 2 "" H 6100 6700 60  0000 C CNN
@@
 Vcap
 $Comp
-L +3V3 #PWR063
+L +3V3 #PWR066
 U 1 1 550F4674
 P 9100 5650
-F 0 "#PWR063" H 9100 5500 60  0001 C CNN
+F 0 "#PWR066" H 9100 5500 60  0001 C CNN
 F 1 "+3V3" H 9100 5790 60  0000 C CNN
 F 2 "" H 9100 5650 60  0000 C CNN
@@
 $EndComp
 $Comp
-L GND #PWR064
+L GND #PWR067
 U 1 1 550F46C2
 P 9100 5800
-F 0 "#PWR064" H 9100 5550 60  0001 C CNN
+F 0 "#PWR067" H 9100 5550 60  0001 C CNN
 F 1 "GND" H 9100 5650 60  0000 C CNN
 F 2 "" H 9100 5800 60  0000 C CNN
@@
 $EndComp
 $Comp
-L GND #PWR065
+L GND #PWR068
 U 1 1 551050BF
 P 9900 3650
-F 0 "#PWR065" H 9900 3400 60  0001 C CNN
+F 0 "#PWR068" H 9900 3400 60  0001 C CNN
 F 1 "GND" H 9900 3500 60  0000 C CNN
 F 2 "" H 9900 3650 60  0000 C CNN
@@
 MCLR_in
 $Comp
-L +3V3 #PWR066
+L +3V3 #PWR069
 U 1 1 5510573C
 P 9700 1750
-F 0 "#PWR066" H 9700 1600 60  0001 C CNN
+F 0 "#PWR069" H 9700 1600 60  0001 C CNN
 F 1 "+3V3" H 9700 1890 60  0000 C CNN
 F 2 "" H 9700 1750 60  0000 C CNN
@@
 $EndComp
 $Comp
-L GND #PWR067
+L GND #PWR070
 U 1 1 55105A71
 P 9350 3050
-F 0 "#PWR067" H 9350 2800 60  0001 C CNN
+F 0 "#PWR070" H 9350 2800 60  0001 C CNN
 F 1 "GND" H 9350 2900 60  0000 C CNN
 F 2 "" H 9350 3050 60  0000 C CNN
@@
 	3550 6200 3550 6250
 $Comp
-L GND #PWR068
+L GND #PWR071
 U 1 1 5513A6E9
 P 3550 6250
-F 0 "#PWR068" H 3550 6000 60  0001 C CNN
+F 0 "#PWR071" H 3550 6000 60  0001 C CNN
 F 1 "GND" H 3550 6100 60  0000 C CNN
 F 2 "" H 3550 6250 60  0000 C CNN

Commit message: Added crystal footprint
Signed-off-by: Kolijn Wolfaardt <kolijn.wolfaardt@gmail.com>
Parts:
- X2: footprint (none) -> RoBoC:Crystal 6x 3.5 x 1.1mm
Changed lines of the file:
@@
 $EndComp
 $Comp
-L +3V3 #PWR053
+L +3V3 #PWR59
 U 1 1 550F44AC
 P 2400 6150
-F 0 "#PWR053" H 2400 6000 60  0001 C CNN
+F 0 "#PWR59" H 2400 6000 60  0001 C CNN
 F 1 "+3V3" H 2400 6290 60  0000 C CNN
 F 2 "" H 2400 6150 60  0000 C CNN
@@
 $EndComp
 $Comp
-L GND #PWR054
+L GND #PWR60
 U 1 1 550F44B3
 P 2400 6450
-F 0 "#PWR054" H 2400 6200 60  0001 C CNN
+F 0 "#PWR60" H 2400 6200 60  0001 C CNN
 F 1 "GND" H 2400 6300 60  0000 C CNN
 F 2 "" H 2400 6450 60  0000 C CNN
@@
 MCLR_in
 $Comp
-L +3V3 #PWR055
+L +3V3 #PWR58
 U 1 1 550F44C2
 P 2250 3700
-F 0 "#PWR055" H 2250 3550 60  0001 C CNN
+F 0 "#PWR58" H 2250 3550 60  0001 C CNN
 F 1 "+3V3" H 2250 3840 60  0000 C CNN
 F 2 "" H 2250 3700 60  0000 C CNN
@@
 $EndComp
 $Comp
-L GND #PWR056
+L GND #PWR54
 U 1 1 550F44C8
 P 2000 4350
-F 0 "#PWR056" H 2000 4100 60  0001 C CNN
+F 0 "#PWR54" H 2000 4100 60  0001 C CNN
 F 1 "GND" H 2000 4200 60  0000 C CNN
 F 2 "" H 2000 4350 60  0000 C CNN
@@
 $EndComp
 $Comp
-L +3V3 #PWR057
+L +3V3 #PWR57
 U 1 1 550F44D2
 P 2200 2000
-F 0 "#PWR057" H 2200 1850 60  0001 C CNN
+F 0 "#PWR57" H 2200 1850 60  0001 C CNN
 F 1 "+3V3" H 2200 2140 60  0000 C CNN
 F 2 "" H 2200 2000 60  0000 C CNN
@@
 $EndComp
 $Comp
-L GND #PWR058
+L GND #PWR53
 U 1 1 550F44D8
 P 2000 2650
-F 0 "#PWR058" H 2000 2400 60  0001 C CNN
+F 0 "#PWR53" H 2000 2400 60  0001 C CNN
 F 1 "GND" H 2000 2500 60  0000 C CNN
 F 2 "" H 2000 2650 60  0000 C CNN
@@
 $EndComp
 $Comp
-L +3V3 #PWR059
+L +3V3 #PWR66
 U 1 1 550F44E2
 P 8000 3950
-F 0 "#PWR059" H 8000 3800 60  0001 C CNN
+F 0 "#PWR66" H 8000 3800 60  0001 C CNN
 F 1 "+3V3" H 8000 4090 60  0000 C CNN
 F 2 "" H 8000 3950 60  0000 C CNN
@@
 $EndComp
 $Comp
-L GND #PWR060
+L GND #PWR64
 U 1 1 550F44E8
 P 7800 3700
-F 0 "#PWR060" H 7800 3450 60  0001 C CNN
+F 0 "#PWR64" H 7800 3450 60  0001 C CNN
 F 1 "GND" H 7800 3550 60  0000 C CNN
 F 2 "" H 7800 3700 60  0000 C CNN
@@
 $EndComp
 $Comp
-L +3V3 #PWR061
+L +3V3 #PWR65
 U 1 1 550F44F1
 P 7850 1900
-F 0 "#PWR061" H 7850 1750 60  0001 C CNN
+F 0 "#PWR65" H 7850 1750 60  0001 C CNN
 F 1 "+3V3" H 7850 2040 60  0000 C CNN
 F 2 "" H 7850 1900 60  0000 C CNN
@@
 PGC
 $Comp
-L +3V3 #PWR062
+L +3V3 #PWR55
 U 1 1 550F450D
 P 2100 3100
-F 0 "#PWR062" H 2100 2950 60  0001 C CNN
+F 0 "#PWR55" H 2100 2950 60  0001 C CNN
 F 1 "+3V3" H 2100 3240 60  0000 C CNN
 F 2 "" H 2100 3100 60  0000 C CNN
@@
 $EndComp
 $Comp
-L GND #PWR063
+L GND #PWR56
 U 1 1 550F4513
 P 2100 3350
-F 0 "#PWR063" H 2100 3100 60  0001 C CNN
+F 0 "#PWR56" H 2100 3100 60  0001 C CNN
 F 1 "GND" H 2100 3200 60  0000 C CNN
 F 2 "" H 2100 3350 60  0000 C CNN
@@
 F 0 "X2" H 3950 6290 50  0000 C CNN
 F 1 "10MHz" H 3980 6090 50  0000 L CNN
-F 2 "" H 3950 6200 60  0001 C CNN
+F 2 "RoBoC:Crystal 6x 3.5 x 1.1mm" H 3950 6200 60  0001 C CNN
 F 3 "" H 3950 6200 60  0000 C CNN
 	1    3950 6200
@@
 $EndComp
 $Comp
-L GND #PWR064
+L GND #PWR62
 U 1 1 550F453B
 P 4550 6600
-F 0 "#PWR064" H 4550 6350 60  0001 C CNN
+F 0 "#PWR62" H 4550 6350 60  0001 C CNN
 F 1 "GND" H 4550 6450 60  0000 C CNN
 F 2 "" H 4550 6600 60  0000 C CNN
@@
 $EndComp
 $Comp
-L GND #PWR065
+L GND #PWR63
 U 1 1 550F4558
 P 6100 6700
-F 0 "#PWR065" H 6100 6450 60  0001 C CNN
+F 0 "#PWR63" H 6100 6450 60  0001 C CNN
 F 1 "GND" H 6100 6550 60  0000 C CNN
 F 2 "" H 6100 6700 60  0000 C CNN
@@
 Vcap
 $Comp
-L +3V3 #PWR066
+L +3V3 #PWR67
 U 1 1 550F4674
 P 9100 5650
-F 0 "#PWR066" H 9100 5500 60  0001 C CNN
+F 0 "#PWR67" H 9100 5500 60  0001 C CNN
 F 1 "+3V3" H 9100 5790 60  0000 C CNN
 F 2 "" H 9100 5650 60  0000 C CNN
@@
 $EndComp
 $Comp
-L GND #PWR067
+L GND #PWR68
 U 1 1 550F46C2
 P 9100 5800
-F 0 "#PWR067" H 9100 5550 60  0001 C CNN
+F 0 "#PWR68" H 9100 5550 60  0001 C CNN
 F 1 "GND" H 9100 5650 60  0000 C CNN
 F 2 "" H 9100 5800 60  0000 C CNN
@@
 $EndComp
 $Comp
-L GND #PWR068
+L GND #PWR71
 U 1 1 551050BF
 P 9900 3650
-F 0 "#PWR068" H 9900 3400 60  0001 C CNN
+F 0 "#PWR71" H 9900 3400 60  0001 C CNN
 F 1 "GND" H 9900 3500 60  0000 C CNN
 F 2 "" H 9900 3650 60  0000 C CNN
@@
 MCLR_in
 $Comp
-L +3V3 #PWR069
+L +3V3 #PWR70
 U 1 1 5510573C
 P 9700 1750
-F 0 "#PWR069" H 9700 1600 60  0001 C CNN
+F 0 "#PWR70" H 9700 1600 60  0001 C CNN
 F 1 "+3V3" H 9700 1890 60  0000 C CNN
 F 2 "" H 9700 1750 60  0000 C CNN
@@
 $EndComp
 $Comp
-L GND #PWR070
+L GND #PWR69
 U 1 1 55105A71
 P 9350 3050
-F 0 "#PWR070" H 9350 2800 60  0001 C CNN
+F 0 "#PWR69" H 9350 2800 60  0001 C CNN
 F 1 "GND" H 9350 2900 60  0000 C CNN
 F 2 "" H 9350 3050 60  0000 C CNN
@@
 	3550 6200 3550 6250
 $Comp
-L GND #PWR071
+L GND #PWR61
 U 1 1 5513A6E9
 P 3550 6250
-F 0 "#PWR071" H 3550 6000 60  0001 C CNN
+F 0 "#PWR61" H 3550 6000 60  0001 C CNN
 F 1 "GND" H 3550 6100 60  0000 C CNN
 F 2 "" H 3550 6250 60  0000 C CNN

Commit message: Finished the footprint allocation, started on the PCB layout.-s
Parts:
- C18, C19: value 22pF -> 12pF
- P14: value CONN_01X06 -> ICSP
Changed lines of the file:
@@
 P 1600 6400
 F 0 "P14" H 1600 6750 50  0000 C CNN
-F 1 "CONN_01X06" V 1700 6400 50  0000 C CNN
+F 1 "ICSP" V 1700 6400 50  0000 C CNN
 F 2 "Pin_Headers:Pin_Header_Straight_1x06" H 1600 6400 60  0001 C CNN
 F 3 "" H 1600 6400 60  0000 C CNN
@@
 $EndComp
 $Comp
-L +3V3 #PWR59
+L +3V3 #PWR053
 U 1 1 550F44AC
 P 2400 6150
-F 0 "#PWR59" H 2400 6000 60  0001 C CNN
+F 0 "#PWR053" H 2400 6000 60  0001 C CNN
 F 1 "+3V3" H 2400 6290 60  0000 C CNN
 F 2 "" H 2400 6150 60  0000 C CNN
@@
 $EndComp
 $Comp
-L GND #PWR60
+L GND #PWR054
 U 1 1 550F44B3
 P 2400 6450
-F 0 "#PWR60" H 2400 6200 60  0001 C CNN
+F 0 "#PWR054" H 2400 6200 60  0001 C CNN
 F 1 "GND" H 2400 6300 60  0000 C CNN
 F 2 "" H 2400 6450 60  0000 C CNN
@@
 MCLR_in
 $Comp
-L +3V3 #PWR58
+L +3V3 #PWR055
 U 1 1 550F44C2
 P 2250 3700
-F 0 "#PWR58" H 2250 3550 60  0001 C CNN
+F 0 "#PWR055" H 2250 3550 60  0001 C CNN
 F 1 "+3V3" H 2250 3840 60  0000 C CNN
 F 2 "" H 2250 3700 60  0000 C CNN
@@
 $EndComp
 $Comp
-L GND #PWR54
+L GND #PWR056
 U 1 1 550F44C8
 P 2000 4350
-F 0 "#PWR54" H 2000 4100 60  0001 C CNN
+F 0 "#PWR056" H 2000 4100 60  0001 C CNN
 F 1 "GND" H 2000 4200 60  0000 C CNN
 F 2 "" H 2000 4350 60  0000 C CNN
@@
 $EndComp
 $Comp
-L +3V3 #PWR57
+L +3V3 #PWR057
 U 1 1 550F44D2
 P 2200 2000
-F 0 "#PWR57" H 2200 1850 60  0001 C CNN
+F 0 "#PWR057" H 2200 1850 60  0001 C CNN
 F 1 "+3V3" H 2200 2140 60  0000 C CNN
 F 2 "" H 2200 2000 60  0000 C CNN
@@
 $EndComp
 $Comp
-L GND #PWR53
+L GND #PWR058
 U 1 1 550F44D8
 P 2000 2650
-F 0 "#PWR53" H 2000 2400 60  0001 C CNN
+F 0 "#PWR058" H 2000 2400 60  0001 C CNN
 F 1 "GND" H 2000 2500 60  0000 C CNN
 F 2 "" H 2000 2650 60  0000 C CNN
@@
 $EndComp
 $Comp
-L +3V3 #PWR66
+L +3V3 #PWR059
 U 1 1 550F44E2
 P 8000 3950
-F 0 "#PWR66" H 8000 3800 60  0001 C CNN
+F 0 "#PWR059" H 8000 3800 60  0001 C CNN
 F 1 "+3V3" H 8000 4090 60  0000 C CNN
 F 2 "" H 8000 3950 60  0000 C CNN
@@
 $EndComp
 $Comp
-L GND #PWR64
+L GND #PWR060
 U 1 1 550F44E8
 P 7800 3700
-F 0 "#PWR64" H 7800 3450 60  0001 C CNN
+F 0 "#PWR060" H 7800 3450 60  0001 C CNN
 F 1 "GND" H 7800 3550 60  0000 C CNN
 F 2 "" H 7800 3700 60  0000 C CNN
@@
 $EndComp
 $Comp
-L +3V3 #PWR65
+L +3V3 #PWR061
 U 1 1 550F44F1
 P 7850 1900
-F 0 "#PWR65" H 7850 1750 60  0001 C CNN
+F 0 "#PWR061" H 7850 1750 60  0001 C CNN
 F 1 "+3V3" H 7850 2040 60  0000 C CNN
 F 2 "" H 7850 1900 60  0000 C CNN
@@
 PGC
 $Comp
-L +3V3 #PWR55
+L +3V3 #PWR062
 U 1 1 550F450D
 P 2100 3100
-F 0 "#PWR55" H 2100 2950 60  0001 C CNN
+F 0 "#PWR062" H 2100 2950 60  0001 C CNN
 F 1 "+3V3" H 2100 3240 60  0000 C CNN
 F 2 "" H 2100 3100 60  0000 C CNN
@@
 $EndComp
 $Comp
-L GND #PWR56
+L GND #PWR063
 U 1 1 550F4513
 P 2100 3350
-F 0 "#PWR56" H 2100 3100 60  0001 C CNN
+F 0 "#PWR063" H 2100 3100 60  0001 C CNN
 F 1 "GND" H 2100 3200 60  0000 C CNN
 F 2 "" H 2100 3350 60  0000 C CNN
@@
 P 4250 5900
 F 0 "C18" H 4300 6000 50  0000 L CNN
-F 1 "22pF" H 4300 5800 50  0000 L CNN
+F 1 "12pF" H 4300 5800 50  0000 L CNN
 F 2 "Capacitors_SMD:C_1206" H 4288 5750 30  0001 C CNN
 F 3 "" H 4250 5900 60  0000 C CNN
@@
 P 4250 6500
 F 0 "C19" H 4300 6600 50  0000 L CNN
-F 1 "22pF" H 4300 6400 50  0000 L CNN
+F 1 "12pF" H 4300 6400 50  0000 L CNN
 F 2 "Capacitors_SMD:C_1206" H 4288 6350 30  0001 C CNN
 F 3 "" H 4250 6500 60  0000 C CNN
@@
 $EndComp
 $Comp
-L GND #PWR62
+L GND #PWR064
 U 1 1 550F453B
 P 4550 6600
-F 0 "#PWR62" H 4550 6350 60  0001 C CNN
+F 0 "#PWR064" H 4550 6350 60  0001 C CNN
 F 1 "GND" H 4550 6450 60  0000 C CNN
 F 2 "" H 4550 6600 60  0000 C CNN
@@
 $EndComp
 $Comp
-L GND #PWR63
+L GND #PWR065
 U 1 1 550F4558
 P 6100 6700
-F 0 "#PWR63" H 6100 6450 60  0001 C CNN
+F 0 "#PWR065" H 6100 6450 60  0001 C CNN
 F 1 "GND" H 6100 6550 60  0000 C CNN
 F 2 "" H 6100 6700 60  0000 C CNN
@@
 Vcap
 $Comp
-L +3V3 #PWR67
+L +3V3 #PWR066
 U 1 1 550F4674
 P 9100 5650
-F 0 "#PWR67" H 9100 5500 60  0001 C CNN
+F 0 "#PWR066" H 9100 5500 60  0001 C CNN
 F 1 "+3V3" H 9100 5790 60  0000 C CNN
 F 2 "" H 9100 5650 60  0000 C CNN
@@
 $EndComp
 $Comp
-L GND #PWR68
+L GND #PWR067
 U 1 1 550F46C2
 P 9100 5800
-F 0 "#PWR68" H 9100 5550 60  0001 C CNN
+F 0 "#PWR067" H 9100 5550 60  0001 C CNN
 F 1 "GND" H 9100 5650 60  0000 C CNN
 F 2 "" H 9100 5800 60  0000 C CNN
@@
 $EndComp
 $Comp
-L GND #PWR71
+L GND #PWR068
 U 1 1 551050BF
 P 9900 3650
-F 0 "#PWR71" H 9900 3400 60  0001 C CNN
+F 0 "#PWR068" H 9900 3400 60  0001 C CNN
 F 1 "GND" H 9900 3500 60  0000 C CNN
 F 2 "" H 9900 3650 60  0000 C CNN
@@
 MCLR_in
 $Comp
-L +3V3 #PWR70
+L +3V3 #PWR069
 U 1 1 5510573C
 P 9700 1750
-F 0 "#PWR70" H 9700 1600 60  0001 C CNN
+F 0 "#PWR069" H 9700 1600 60  0001 C CNN
 F 1 "+3V3" H 9700 1890 60  0000 C CNN
 F 2 "" H 9700 1750 60  0000 C CNN
@@
 $EndComp
 $Comp
-L GND #PWR69
+L GND #PWR070
 U 1 1 55105A71
 P 9350 3050
-F 0 "#PWR69" H 9350 2800 60  0001 C CNN
+F 0 "#PWR070" H 9350 2800 60  0001 C CNN
 F 1 "GND" H 9350 2900 60  0000 C CNN
 F 2 "" H 9350 3050 60  0000 C CNN
@@
 	3550 6200 3550 6250
 $Comp
-L GND #PWR61
+L GND #PWR071
 U 1 1 5513A6E9
 P 3550 6250
-F 0 "#PWR61" H 3550 6000 60  0001 C CNN
+F 0 "#PWR071" H 3550 6000 60  0001 C CNN
 F 1 "GND" H 3550 6100 60  0000 C CNN
 F 2 "" H 3550 6250 60  0000 C CNN

Commit message: Added UART, Gnd and 3.3v pins
Signed-off-by: Kolijn Wolfaardt <kolijn.wolfaardt@gmail.com>
Parts:
- added P?: UART, symbol CONN_01X03
Connections:
- wire segments 103 -> 115
Changed lines of the file:
@@
 	2950 1900 3400 1900
 Wire Wire Line
-	4550 5900 4550 6600
+	4550 5900 4550 6500
+Wire Wire Line
+	4550 6500 4550 6600
 Wire Wire Line
 	4400 5900 4550 5900
@@
 	3950 6400 3950 6500
 Wire Wire Line
-	3350 6500 4100 6500
+	3350 6500 3950 6500
+Wire Wire Line
+	3950 6500 4100 6500
 Connection ~ 3950 6500
 Wire Wire Line
-	3350 5900 4100 5900
+	3350 5900 3950 5900
+Wire Wire Line
+	3950 5900 4100 5900
 Wire Wire Line
 	3950 6000 3950 5900
@@
 	9700 3550 9700 3650
 Wire Wire Line
-	9700 3650 10100 3650
+	9700 3650 9900 3650
+Wire Wire Line
+	9900 3650 10100 3650
 Wire Wire Line
 	10100 3650 10100 3550
 Connection ~ 9900 3650
 Wire Wire Line
-	9100 2450 10600 2450
-Wire Wire Line
-	9700 2250 9700 2550
+	9100 2450 9350 2450
+Wire Wire Line
+	9350 2450 9700 2450
+Wire Wire Line
+	9700 2450 10100 2450
+Wire Wire Line
+	10100 2450 10600 2450
+Wire Wire Line
+	9700 2250 9700 2450
+Wire Wire Line
+	9700 2450 9700 2550
 Connection ~ 9700 2450
 Wire Wire Line
@@
 NoConn ~ 7150 1800
 NoConn ~ 7150 1900
+$Comp
+L CONN_01X03 P?
+U 1 1 551D06D3
+P 9700 4650
+F 0 "P?" H 9700 4850 50  0000 C CNN
+F 1 "UART" V 9800 4650 50  0000 C CNN
+F 2 "" H 9700 4650 60  0000 C CNN
+F 3 "" H 9700 4650 60  0000 C CNN
+	1    9700 4650
+	1    0    0    -1
+$EndComp
+Text HLabel 9400 4550 0    60   Input ~ 0
+U1RX
+Text HLabel 9400 4750 0    60   Output ~ 0
+U1TX
+$Comp
+L GND #PWR?
+U 1 1 551D07D4
+P 8950 4700
+F 0 "#PWR?" H 8950 4450 60  0001 C CNN
+F 1 "GND" H 8950 4550 60  0000 C CNN
+F 2 "" H 8950 4700 60  0000 C CNN
+F 3 "" H 8950 4700 60  0000 C CNN
+	1    8950 4700
+	1    0    0    -1
+$EndComp
+Wire Wire Line
+	8950 4700 8950 4650
+Wire Wire Line
+	8950 4650 9500 4650
+Wire Wire Line
+	9500 4550 9400 4550
+Wire Wire Line
+	9400 4750 9500 4750
 $EndSCHEMATC
