File: PCB Design/mcu.sch (KiCad schematic (older format))
At the start: 11 parts, among them P14 ICSP, P16 UART, U4 dsPIC33FJ32GS606, X2 10MHz

Commit message: Increased pad sizes for easy soldering, final commit before ordering
Signed-off-by: Kolijn Wolfaardt <kolijn.wolfaardt@gmail.com>
Parts:
- RESET1: footprint Buttons_Switches_SMD:SW_SPST_PTS645 -> RoBoC:SW_SPST_bigpads
- U4: footprint Housings_QFP:TQFP-64_10x10mm_Pitch0.5mm -> RoBoC:TQFP-64_10x10mm_Pitch0.5mm_handsoldering
Changed lines of the file:
@@
 F 0 "U4" H 5200 3650 60  0000 C CNN
 F 1 "dsPIC33FJ32GS606" H 5150 150 60  0000 C CNN
-F 2 "Housings_QFP:TQFP-64_10x10mm_Pitch0.5mm" H 5200 2400 60  0001 C CNN
+F 2 "RoBoC:TQFP-64_10x10mm_Pitch0.5mm_handsoldering" H 5200 2400 60  0001 C CNN
 F 3 "" H 5200 2400 60  0000 C CNN
 	1    5200 2400
@@
 F 0 "RESET1" H 10200 3100 50  0000 C CNN
 F 1 "DPST" H 10200 3000 50  0000 C CNN
-F 2 "Buttons_Switches_SMD:SW_SPST_PTS645" H 9900 3050 60  0001 C CNN
+F 2 "RoBoC:SW_SPST_bigpads" H 9900 3050 60  0001 C CNN
 F 3 "" H 9900 3050 60  0000 C CNN
 	1    9900 3050
