File: PCB Design/gpio.sch (KiCad schematic (older format))
At the start: 25 parts, among them P10 CONN_02X11, P11 CONN_01X03, P12 CONN_01X02, P13 CONN_01X06, P9 CONN_01X08, SW0 DPST, SW1 DPST

Commit message: Added initial footprint associations, caps and resistors.
Kicad is giving weird errors for the libraries and BOM generator.
The libraries have to be downloaded manually from github, and
then added.

Signed-off-by: Kolijn Wolfaardt <kolijn.wolfaardt@gmail.com>
Parts:
- C12, C13, C14: footprint (none) -> Capacitors_SMD:C_1206
- D1, D2, D3, D4, D5, D6: footprint (none) -> LEDs:LED-1206
- P10: footprint (none) -> Pin_Headers:Pin_Header_Straight_2x11
- P11: footprint (none) -> Pin_Headers:Pin_Header_Straight_1x03
- P12: footprint (none) -> Pin_Headers:Pin_Header_Straight_1x02
- P13: footprint (none) -> Pin_Headers:Pin_Header_Straight_1x06
- P9: footprint (none) -> Pin_Headers:Pin_Header_Straight_1x08
- R1, R2, R3, R4, R5, R6, R7, R8, R9: footprint (none) -> Resistors_SMD:R_1206
- SW0, SW1: footprint (none) -> Buttons_Switches_SMD:SW_SPST_PTS645
Changed lines of the file:
@@
 F 0 "D2" H 1950 3600 50  0000 C CNN
 F 1 "LED" H 1950 3400 50  0000 C CNN
-F 2 "" H 1950 3500 60  0000 C CNN
+F 2 "LEDs:LED-1206" H 1950 3500 60  0001 C CNN
 F 3 "" H 1950 3500 60  0000 C CNN
 	1    1950 3500
@@
 F 0 "D3" H 2250 3600 50  0000 C CNN
 F 1 "LED" H 2250 3400 50  0000 C CNN
-F 2 "" H 2250 3500 60  0000 C CNN
+F 2 "LEDs:LED-1206" H 2250 3500 60  0001 C CNN
 F 3 "" H 2250 3500 60  0000 C CNN
 	1    2250 3500
@@
 F 0 "D4" H 2550 3600 50  0000 C CNN
 F 1 "LED" H 2550 3400 50  0000 C CNN
-F 2 "" H 2550 3500 60  0000 C CNN
+F 2 "LEDs:LED-1206" H 2550 3500 60  0001 C CNN
 F 3 "" H 2550 3500 60  0000 C CNN
 	1    2550 3500
@@
 F 0 "D5" H 2850 3600 50  0000 C CNN
 F 1 "LED" H 2850 3400 50  0000 C CNN
-F 2 "" H 2850 3500 60  0000 C CNN
+F 2 "LEDs:LED-1206" H 2850 3500 60  0001 C CNN
 F 3 "" H 2850 3500 60  0000 C CNN
 	1    2850 3500
@@
 F 0 "D6" H 3150 3600 50  0000 C CNN
 F 1 "LED" H 3150 3400 50  0000 C CNN
-F 2 "" H 3150 3500 60  0000 C CNN
+F 2 "LEDs:LED-1206" H 3150 3500 60  0001 C CNN
 F 3 "" H 3150 3500 60  0000 C CNN
 	1    3150 3500
@@
 F 0 "R3" V 2030 4050 50  0000 C CNN
 F 1 "220" V 1957 4051 50  0000 C CNN
-F 2 "" V 1880 4050 30  0000 C CNN
+F 2 "Resistors_SMD:R_1206" V 1880 4050 30  0001 C CNN
 F 3 "" H 1950 4050 30  0000 C CNN
 	1    1950 4050
@@
 F 0 "R4" V 2330 4050 50  0000 C CNN
 F 1 "220" V 2257 4051 50  0000 C CNN
-F 2 "" V 2180 4050 30  0000 C CNN
+F 2 "Resistors_SMD:R_1206" V 2180 4050 30  0001 C CNN
 F 3 "" H 2250 4050 30  0000 C CNN
 	1    2250 4050
@@
 F 0 "R5" V 2630 4050 50  0000 C CNN
 F 1 "220" V 2557 4051 50  0000 C CNN
-F 2 "" V 2480 4050 30  0000 C CNN
+F 2 "Resistors_SMD:R_1206" V 2480 4050 30  0001 C CNN
 F 3 "" H 2550 4050 30  0000 C CNN
 	1    2550 4050
@@
 F 0 "R6" V 2930 4050 50  0000 C CNN
 F 1 "220" V 2857 4051 50  0000 C CNN
-F 2 "" V 2780 4050 30  0000 C CNN
+F 2 "Resistors_SMD:R_1206" V 2780 4050 30  0001 C CNN
 F 3 "" H 2850 4050 30  0000 C CNN
 	1    2850 4050
@@
 F 0 "R8" V 3230 4050 50  0000 C CNN
 F 1 "220" V 3157 4051 50  0000 C CNN
-F 2 "" V 3080 4050 30  0000 C CNN
+F 2 "Resistors_SMD:R_1206" V 3080 4050 30  0001 C CNN
 F 3 "" H 3150 4050 30  0000 C CNN
 	1    3150 4050
@@
 F 0 "SW0" H 2150 6600 50  0000 C CNN
 F 1 "DPST" H 2150 6500 50  0000 C CNN
-F 2 "" H 1850 6550 60  0000 C CNN
+F 2 "Buttons_Switches_SMD:SW_SPST_PTS645" H 1850 6550 60  0001 C CNN
 F 3 "" H 1850 6550 60  0000 C CNN
 	1    1850 6550
@@
 F 0 "R2" V 1730 5650 50  0000 C CNN
 F 1 "4.7k" V 1657 5651 50  0000 C CNN
-F 2 "" V 1580 5650 30  0000 C CNN
+F 2 "Resistors_SMD:R_1206" V 1580 5650 30  0001 C CNN
 F 3 "" H 1650 5650 30  0000 C CNN
 	1    1650 5650
@@
 F 0 "SW1" H 3600 6600 50  0000 C CNN
 F 1 "DPST" H 3600 6500 50  0000 C CNN
-F 2 "" H 3300 6550 60  0000 C CNN
+F 2 "Buttons_Switches_SMD:SW_SPST_PTS645" H 3300 6550 60  0001 C CNN
 F 3 "" H 3300 6550 60  0000 C CNN
 	1    3300 6550
@@
 F 0 "R7" V 3180 5650 50  0000 C CNN
 F 1 "4.7k" V 3107 5651 50  0000 C CNN
-F 2 "" V 3030 5650 30  0000 C CNN
+F 2 "Resistors_SMD:R_1206" V 3030 5650 30  0001 C CNN
 F 3 "" H 3100 5650 30  0000 C CNN
 	1    3100 5650
@@
 F 0 "P10" H 5500 4100 50  0000 C CNN
 F 1 "CONN_02X11" V 5500 3500 50  0000 C CNN
-F 2 "" H 5500 2300 60  0000 C CNN
+F 2 "Pin_Headers:Pin_Header_Straight_2x11" H 5500 2300 60  0001 C CNN
 F 3 "" H 5500 2300 60  0000 C CNN
 	1    5500 3500
@@
 F 0 "P13" H 9400 3900 50  0000 C CNN
 F 1 "CONN_01X06" V 9500 3550 50  0000 C CNN
-F 2 "" H 9400 3550 60  0000 C CNN
+F 2 "Pin_Headers:Pin_Header_Straight_1x06" H 9400 3550 60  0001 C CNN
 F 3 "" H 9400 3550 60  0000 C CNN
 	1    9400 3550
@@
 F 0 "P11" H 6100 5800 50  0000 C CNN
 F 1 "CONN_01X03" V 6200 5600 50  0000 C CNN
-F 2 "" H 6100 5600 60  0000 C CNN
+F 2 "Pin_Headers:Pin_Header_Straight_1x03" H 6100 5600 60  0001 C CNN
 F 3 "" H 6100 5600 60  0000 C CNN
 	1    6100 5600
@@
 F 0 "D1" H 1650 3600 50  0000 C CNN
 F 1 "LED" H 1650 3400 50  0000 C CNN
-F 2 "" H 1650 3500 60  0000 C CNN
+F 2 "LEDs:LED-1206" H 1650 3500 60  0001 C CNN
 F 3 "" H 1650 3500 60  0000 C CNN
 	1    1650 3500
@@
 F 0 "R1" V 1730 4050 50  0000 C CNN
 F 1 "220" V 1657 4051 50  0000 C CNN
-F 2 "" V 1580 4050 30  0000 C CNN
+F 2 "Resistors_SMD:R_1206" V 1580 4050 30  0001 C CNN
 F 3 "" H 1650 4050 30  0000 C CNN
 	1    1650 4050
@@
 F 0 "P9" H 2050 1700 50  0000 C CNN
 F 1 "CONN_01X08" V 2150 1250 50  0000 C CNN
-F 2 "" H 2050 1250 60  0000 C CNN
+F 2 "Pin_Headers:Pin_Header_Straight_1x08" H 2050 1250 60  0001 C CNN
 F 3 "" H 2050 1250 60  0000 C CNN
 	1    2050 1250
@@
 F 0 "C12" H 1450 6650 50  0000 L CNN
 F 1 "10nF" H 1450 6450 50  0000 L CNN
-F 2 "" H 1438 6400 30  0000 C CNN
+F 2 "Capacitors_SMD:C_1206" H 1438 6400 30  0001 C CNN
 F 3 "" H 1400 6550 60  0000 C CNN
 	1    1400 6550
@@
 F 0 "C13" H 2900 6650 50  0000 L CNN
 F 1 "10nF" H 2900 6450 50  0000 L CNN
-F 2 "" H 2888 6400 30  0000 C CNN
+F 2 "Capacitors_SMD:C_1206" H 2888 6400 30  0001 C CNN
 F 3 "" H 2850 6550 60  0000 C CNN
 	1    2850 6550
@@
 F 0 "P12" H 8650 5800 50  0000 C CNN
 F 1 "CONN_01X02" V 8750 5650 50  0000 C CNN
-F 2 "" H 8650 5650 60  0000 C CNN
+F 2 "Pin_Headers:Pin_Header_Straight_1x02" H 8650 5650 60  0001 C CNN
 F 3 "" H 8650 5650 60  0000 C CNN
 	1    8650 5650
@@
 F 0 "R9" V 8380 5300 50  0000 C CNN
 F 1 "4.7k" V 8307 5301 50  0000 C CNN
-F 2 "" V 8230 5300 30  0000 C CNN
+F 2 "Resistors_SMD:R_1206" V 8230 5300 30  0001 C CNN
 F 3 "" H 8300 5300 30  0000 C CNN
 	1    8300 5300
@@
 F 0 "C14" H 8000 5900 50  0000 L CNN
 F 1 "10nF" H 8000 5700 50  0000 L CNN
-F 2 "" H 7988 5650 30  0000 C CNN
+F 2 "Capacitors_SMD:C_1206" H 7988 5650 30  0001 C CNN
 F 3 "" H 7950 5800 60  0000 C CNN
 	1    7950 5800

Commit message: Finished the footprint allocation, started on the PCB layout.-s
Parts:
- D1: value LED -> LED5
- D2: value LED -> LED4
- D3: value LED -> LED3
- D4: value LED -> LED2
- D5: value LED -> LED1
- D6: value LED -> LED0
- P10: value CONN_02X11 -> Camera
- P11: value CONN_01X03 -> DAC
- P12: value CONN_01X02 -> Reed
- P13: value CONN_01X06 -> SPI
- P9: value CONN_01X08 -> Analog
- SW0: value DPST -> But 0
- SW1: value DPST -> But 1
Changed lines of the file:
@@
 P 1950 3500
 F 0 "D2" H 1950 3600 50  0000 C CNN
-F 1 "LED" H 1950 3400 50  0000 C CNN
+F 1 "LED4" H 1950 3400 50  0000 C CNN
 F 2 "LEDs:LED-1206" H 1950 3500 60  0001 C CNN
 F 3 "" H 1950 3500 60  0000 C CNN
@@
 P 2250 3500
 F 0 "D3" H 2250 3600 50  0000 C CNN
-F 1 "LED" H 2250 3400 50  0000 C CNN
+F 1 "LED3" H 2250 3400 50  0000 C CNN
 F 2 "LEDs:LED-1206" H 2250 3500 60  0001 C CNN
 F 3 "" H 2250 3500 60  0000 C CNN
@@
 P 2550 3500
 F 0 "D4" H 2550 3600 50  0000 C CNN
-F 1 "LED" H 2550 3400 50  0000 C CNN
+F 1 "LED2" H 2550 3400 50  0000 C CNN
 F 2 "LEDs:LED-1206" H 2550 3500 60  0001 C CNN
 F 3 "" H 2550 3500 60  0000 C CNN
@@
 P 2850 3500
 F 0 "D5" H 2850 3600 50  0000 C CNN
-F 1 "LED" H 2850 3400 50  0000 C CNN
+F 1 "LED1" H 2850 3400 50  0000 C CNN
 F 2 "LEDs:LED-1206" H 2850 3500 60  0001 C CNN
 F 3 "" H 2850 3500 60  0000 C CNN
@@
 P 3150 3500
 F 0 "D6" H 3150 3600 50  0000 C CNN
-F 1 "LED" H 3150 3400 50  0000 C CNN
+F 1 "LED0" H 3150 3400 50  0000 C CNN
 F 2 "LEDs:LED-1206" H 3150 3500 60  0001 C CNN
 F 3 "" H 3150 3500 60  0000 C CNN
@@
 $EndComp
 $Comp
-L +3V3 #PWR32
+L +3V3 #PWR025
 U 1 1 5510863A
 P 3800 1100
-F 0 "#PWR32" H 3800 950 60  0001 C CNN
+F 0 "#PWR025" H 3800 950 60  0001 C CNN
 F 1 "+3V3" H 3800 1240 60  0000 C CNN
 F 2 "" H 3800 1100 60  0000 C CNN
@@
 $EndComp
 $Comp
-L GND #PWR33
+L GND #PWR026
 U 1 1 55108640
 P 3800 1250
-F 0 "#PWR33" H 3800 1000 60  0001 C CNN
+F 0 "#PWR026" H 3800 1000 60  0001 C CNN
 F 1 "GND" H 3800 1100 60  0000 C CNN
 F 2 "" H 3800 1250 60  0000 C CNN
@@
 GND
 $Comp
-L GND #PWR29
+L GND #PWR027
 U 1 1 5510866B
 P 2550 4450
-F 0 "#PWR29" H 2550 4200 60  0001 C CNN
+F 0 "#PWR027" H 2550 4200 60  0001 C CNN
 F 1 "GND" H 2550 4300 60  0000 C CNN
 F 2 "" H 2550 4450 60  0000 C CNN
@@
 P 1850 6550
 F 0 "SW0" H 2150 6600 50  0000 C CNN
-F 1 "DPST" H 2150 6500 50  0000 C CNN
+F 1 "But 0" H 2150 6500 50  0000 C CNN
 F 2 "Buttons_Switches_SMD:SW_SPST_PTS645" H 1850 6550 60  0001 C CNN
 F 3 "" H 1850 6550 60  0000 C CNN
@@
 $EndComp
 $Comp
-L GND #PWR28
+L GND #PWR028
 U 1 1 5510AC8C
 P 1850 7150
-F 0 "#PWR28" H 1850 6900 60  0001 C CNN
+F 0 "#PWR028" H 1850 6900 60  0001 C CNN
 F 1 "GND" H 1850 7000 60  0000 C CNN
 F 2 "" H 1850 7150 60  0000 C CNN
@@
 $EndComp
 $Comp
-L +3V3 #PWR25
+L +3V3 #PWR029
 U 1 1 5510AFD1
 P 1650 5300
-F 0 "#PWR25" H 1650 5150 60  0001 C CNN
+F 0 "#PWR029" H 1650 5150 60  0001 C CNN
 F 1 "+3V3" H 1650 5440 60  0000 C CNN
 F 2 "" H 1650 5300 60  0000 C CNN
@@
 P 3300 6550
 F 0 "SW1" H 3600 6600 50  0000 C CNN
-F 1 "DPST" H 3600 6500 50  0000 C CNN
+F 1 "But 1" H 3600 6500 50  0000 C CNN
 F 2 "Buttons_Switches_SMD:SW_SPST_PTS645" H 3300 6550 60  0001 C CNN
 F 3 "" H 3300 6550 60  0000 C CNN
@@
 $EndComp
 $Comp
-L GND #PWR31
+L GND #PWR030
 U 1 1 5510B4C4
 P 3300 7150
-F 0 "#PWR31" H 3300 6900 60  0001 C CNN
+F 0 "#PWR030" H 3300 6900 60  0001 C CNN
 F 1 "GND" H 3300 7000 60  0000 C CNN
 F 2 "" H 3300 7150 60  0000 C CNN
@@
 $EndComp
 $Comp
-L +3V3 #PWR30
+L +3V3 #PWR031
 U 1 1 5510B4D0
 P 3100 5300
-F 0 "#PWR30" H 3100 5150 60  0001 C CNN
+F 0 "#PWR031" H 3100 5150 60  0001 C CNN
 F 1 "+3V3" H 3100 5440 60  0000 C CNN
 F 2 "" H 3100 5300 60  0000 C CNN
@@
 P 5500 3500
 F 0 "P10" H 5500 4100 50  0000 C CNN
-F 1 "CONN_02X11" V 5500 3500 50  0000 C CNN
+F 1 "Camera" V 5500 3500 50  0000 C CNN
 F 2 "Pin_Headers:Pin_Header_Straight_2x11" H 5500 2300 60  0001 C CNN
 F 3 "" H 5500 2300 60  0000 C CNN
@@
 $EndComp
 $Comp
-L +3V3 #PWR35
+L +3V3 #PWR032
 U 1 1 5511109F
 P 4950 3000
-F 0 "#PWR35" H 4950 2850 60  0001 C CNN
+F 0 "#PWR032" H 4950 2850 60  0001 C CNN
 F 1 "+3V3" H 4950 3140 60  0000 C CNN
 F 2 "" H 4950 3000 60  0000 C CNN
@@
 $EndComp
 $Comp
-L GND #PWR39
+L GND #PWR033
 U 1 1 551110A5
 P 6450 3050
-F 0 "#PWR39" H 6450 2800 60  0001 C CNN
+F 0 "#PWR033" H 6450 2800 60  0001 C CNN
 F 1 "GND" H 6450 2900 60  0000 C CNN
 F 2 "" H 6450 3050 60  0000 C CNN
@@
 SPI_SS
 $Comp
-L +3V3 #PWR42
+L +3V3 #PWR034
 U 1 1 5511AF73
 P 8950 3200
-F 0 "#PWR42" H 8950 3050 60  0001 C CNN
+F 0 "#PWR034" H 8950 3050 60  0001 C CNN
 F 1 "+3V3" H 8950 3340 60  0000 C CNN
 F 2 "" H 8950 3200 60  0000 C CNN
@@
 $EndComp
 $Comp
-L GND #PWR43
+L GND #PWR035
 U 1 1 5511AF79
 P 8950 3850
-F 0 "#PWR43" H 8950 3600 60  0001 C CNN
+F 0 "#PWR035" H 8950 3600 60  0001 C CNN
 F 1 "GND" H 8950 3700 60  0000 C CNN
 F 2 "" H 8950 3850 60  0000 C CNN
@@
 P 9400 3550
 F 0 "P13" H 9400 3900 50  0000 C CNN
-F 1 "CONN_01X06" V 9500 3550 50  0000 C CNN
+F 1 "SPI" V 9500 3550 50  0000 C CNN
 F 2 "Pin_Headers:Pin_Header_Straight_1x06" H 9400 3550 60  0001 C CNN
 F 3 "" H 9400 3550 60  0000 C CNN
@@
 P 6100 5600
 F 0 "P11" H 6100 5800 50  0000 C CNN
-F 1 "CONN_01X03" V 6200 5600 50  0000 C CNN
+F 1 "DAC" V 6200 5600 50  0000 C CNN
 F 2 "Pin_Headers:Pin_Header_Straight_1x03" H 6100 5600 60  0001 C CNN
 F 3 "" H 6100 5600 60  0000 C CNN
@@
 $EndComp
 $Comp
-L GND #PWR37
+L GND #PWR036
 U 1 1 5511E511
 P 5800 5800
-F 0 "#PWR37" H 5800 5550 60  0001 C CNN
+F 0 "#PWR036" H 5800 5550 60  0001 C CNN
 F 1 "GND" H 5800 5650 60  0000 C CNN
 F 2 "" H 5800 5800 60  0000 C CNN
@@
 $EndComp
 $Comp
-L +3V3 #PWR36
+L +3V3 #PWR037
 U 1 1 5511E6AC
 P 5800 5400
-F 0 "#PWR36" H 5800 5250 60  0001 C CNN
+F 0 "#PWR037" H 5800 5250 60  0001 C CNN
 F 1 "+3V3" H 5800 5540 60  0000 C CNN
 F 2 "" H 5800 5400 60  0000 C CNN
@@
 DACOUT
 $Comp
-L GND #PWR41
+L GND #PWR038
 U 1 1 5511FB12
 P 8350 6050
-F 0 "#PWR41" H 8350 5800 60  0001 C CNN
+F 0 "#PWR038" H 8350 5800 60  0001 C CNN
 F 1 "GND" H 8350 5900 60  0000 C CNN
 F 2 "" H 8350 6050 60  0000 C CNN
@@
 $EndComp
 $Comp
-L +3V3 #PWR40
+L +3V3 #PWR039
 U 1 1 5511FB18
 P 8300 4950
-F 0 "#PWR40" H 8300 4800 60  0001 C CNN
+F 0 "#PWR039" H 8300 4800 60  0001 C CNN
 F 1 "+3V3" H 8300 5090 60  0000 C CNN
 F 2 "" H 8300 4950 60  0000 C CNN
@@
 P 1650 3500
 F 0 "D1" H 1650 3600 50  0000 C CNN
-F 1 "LED" H 1650 3400 50  0000 C CNN
+F 1 "LED5" H 1650 3400 50  0000 C CNN
 F 2 "LEDs:LED-1206" H 1650 3500 60  0001 C CNN
 F 3 "" H 1650 3500 60  0000 C CNN
@@
 $EndComp
 $Comp
-L +3V3 #PWR26
+L +3V3 #PWR040
 U 1 1 55118FCE
 P 1700 900
-F 0 "#PWR26" H 1700 750 60  0001 C CNN
+F 0 "#PWR040" H 1700 750 60  0001 C CNN
 F 1 "+3V3" H 1700 1040 60  0000 C CNN
 F 2 "" H 1700 900 60  0000 C CNN
@@
 $EndComp
 $Comp
-L GND #PWR27
+L GND #PWR041
 U 1 1 55118FD4
 P 1700 1650
-F 0 "#PWR27" H 1700 1400 60  0001 C CNN
+F 0 "#PWR041" H 1700 1400 60  0001 C CNN
 F 1 "GND" H 1700 1500 60  0000 C CNN
 F 2 "" H 1700 1650 60  0000 C CNN
@@
 P 2050 1250
 F 0 "P9" H 2050 1700 50  0000 C CNN
-F 1 "CONN_01X08" V 2150 1250 50  0000 C CNN
+F 1 "Analog" V 2150 1250 50  0000 C CNN
 F 2 "Pin_Headers:Pin_Header_Straight_1x08" H 2050 1250 60  0001 C CNN
 F 3 "" H 2050 1250 60  0000 C CNN
@@
 P 8650 5650
 F 0 "P12" H 8650 5800 50  0000 C CNN
-F 1 "CONN_01X02" V 8750 5650 50  0000 C CNN
+F 1 "Reed" V 8750 5650 50  0000 C CNN
 F 2 "Pin_Headers:Pin_Header_Straight_1x02" H 8650 5650 60  0001 C CNN
 F 3 "" H 8650 5650 60  0000 C CNN
@@
 Strobe
 $Comp
-L +3V3 #PWR34
+L +3V3 #PWR042
 U 1 1 551391B0
 P 4600 3650
-F 0 "#PWR34" H 4600 3500 60  0001 C CNN
+F 0 "#PWR042" H 4600 3500 60  0001 C CNN
 F 1 "+3V3" H 4600 3790 60  0000 C CNN
 F 2 "" H 4600 3650 60  0000 C CNN
@@
 	4600 3700 4600 3650
 $Comp
-L GND #PWR38
+L GND #PWR043
 U 1 1 55139944
 P 6400 3800
-F 0 "#PWR38" H 6400 3550 60  0001 C CNN
+F 0 "#PWR043" H 6400 3550 60  0001 C CNN
 F 1 "GND" H 6400 3650 60  0000 C CNN
 F 2 "" H 6400 3800 60  0000 C CNN

Commit message: Added UART, Gnd and 3.3v pins
Signed-off-by: Kolijn Wolfaardt <kolijn.wolfaardt@gmail.com>
Parts:
- added P?: 3.3v, symbol CONN_01X05
- added P?: Gnd, symbol CONN_01X05
Connections:
- net +3V3: now also P?.1 (P1), P?.2 (P2), P?.3 (P3), P?.4 (P4), P?.5 (P5)
- net GND: now also P?.1 (P1), P?.2 (P2), P?.3 (P3), P?.4 (P4), P?.5 (P5)

Commit message: PCB is now 10cmx5cm, some components moved around for more space
Signed-off-by: Kolijn Wolfaardt <kolijn.wolfaardt@gmail.com>
Parts:
- P15, P2: renamed from P?; footprint (none) -> Pin_Headers:Pin_Header_Straight_1x05
Changed lines of the file:
@@
 NoConn ~ 4800 3800
 $Comp
-L CONN_01X05 P?
+L CONN_01X05 P2
 U 1 1 551D10AE
 P 7600 1400
-F 0 "P?" H 7600 1700 50  0000 C CNN
+F 0 "P2" H 7600 1700 50  0000 C CNN
 F 1 "3.3v" V 7700 1400 50  0000 C CNN
-F 2 "" H 7600 1400 60  0000 C CNN
+F 2 "Pin_Headers:Pin_Header_Straight_1x05" H 7600 1400 60  0001 C CNN
 F 3 "" H 7600 1400 60  0000 C CNN
 	1    7600 1400
@@
 $EndComp
 $Comp
-L CONN_01X05 P?
+L CONN_01X05 P15
 U 1 1 551D1127
 P 8400 1400
-F 0 "P?" H 8400 1700 50  0000 C CNN
+F 0 "P15" H 8400 1700 50  0000 C CNN
 F 1 "Gnd" V 8500 1400 50  0000 C CNN
-F 2 "" H 8400 1400 60  0000 C CNN
+F 2 "Pin_Headers:Pin_Header_Straight_1x05" H 8400 1400 60  0001 C CNN
 F 3 "" H 8400 1400 60  0000 C CNN
 	1    8400 1400
@@
 $EndComp
 $Comp
-L GND #PWR?
+L GND #PWR044
 U 1 1 551D1320
 P 8100 1700
-F 0 "#PWR?" H 8100 1450 60  0001 C CNN
+F 0 "#PWR044" H 8100 1450 60  0001 C CNN
 F 1 "GND" H 8100 1550 60  0000 C CNN
 F 2 "" H 8100 1700 60  0000 C CNN
@@
 Connection ~ 8100 1600
 $Comp
-L +3V3 #PWR?
+L +3V3 #PWR045
 U 1 1 551D19F0
 P 7300 1100
-F 0 "#PWR?" H 7300 950 60  0001 C CNN
+F 0 "#PWR045" H 7300 950 60  0001 C CNN
 F 1 "+3V3" H 7300 1240 60  0000 C CNN
 F 2 "" H 7300 1100 60  0000 C CNN

Commit message: Did some fixes, added better footprint for the flyback diodes:
Re-routed camera bus so that there is more ground for the crystal.
Added ground pour keepouts under the MCU.
Changed the footprint for the motor flyback diodes.
Changed the camera module to have 24 pins, 2 won't be connected
Checked the footprints for dsPIC, MCP and LV8045
Increased thermal pad for voltage regulator

Signed-off-by: Kolijn Wolfaardt <kolijn.wolfaardt@gmail.com>
Parts:
- removed P10: Camera, Pin_Headers:Pin_Header_Straight_2x11, symbol CONN_02X11
- added P10: CONN_02X12, Pin_Headers:Pin_Header_Straight_2x12, symbol CONN_02X12
Connections:
- net +3V3: now also P10.1 (P1), P10.15 (P15)
- net DATA_0: now also P10.14 (P14)
- net DATA_1: now also P10.13 (P13)
- net DATA_2: now also P10.12 (P12)
- net DATA_3: now also P10.11 (P11)
- net DATA_4: now also P10.10 (P10)
- net DATA_5: now also P10.9 (P9)
- net DATA_6: now also P10.8 (P8)
- net DATA_7: now also P10.7 (P7)
- net GND: now also P10.16 (P16), P10.2 (P2)
- net Href: now also P10.6 (P6)
- net RCK: now also P10.18 (P18)
- net SIO_C: now also P10.3 (P3)
- net SIO_D: now also P10.4 (P4)
- net Strobe: now also P10.17 (P17)
- net vSync: now also P10.5 (P5)
- net ~OE: now also P10.20 (P20)
- net ~RRST: now also P10.22 (P22)
- net ~WR: now also P10.19 (P19)
- net ~WRST: now also P10.21 (P21)
- no-connect marks 1 -> 3
Changed lines of the file:
@@
 ~RRST
-$Comp
-L CONN_02X11 P10
-U 1 1 55110EFC
-P 5500 3500
-F 0 "P10" H 5500 4100 50  0000 C CNN
-F 1 "Camera" V 5500 3500 50  0000 C CNN
-F 2 "Pin_Headers:Pin_Header_Straight_2x11" H 5500 2300 60  0001 C CNN
-F 3 "" H 5500 2300 60  0000 C CNN
-	1    5500 3500
-	1    0    0    -1
-$EndComp
 $Comp
 L +3V3 #PWR032
@@
 	7300 1600 7400 1600
 Connection ~ 7300 1500
+$Comp
+L CONN_02X12 P10
+U 1 1 5533AE4A
+P 5500 3550
+F 0 "P10" H 5500 4200 50  0000 C CNN
+F 1 "CONN_02X12" V 5500 3550 50  0000 C CNN
+F 2 "Pin_Headers:Pin_Header_Straight_2x12" H 5500 2350 60  0001 C CNN
+F 3 "" H 5500 2350 60  0000 C CNN
+	1    5500 3550
+	1    0    0    -1
+$EndComp
+NoConn ~ 5750 4100
+NoConn ~ 5250 4100
 $EndSCHEMATC

Commit message: Increased pad sizes for easy soldering, final commit before ordering
Signed-off-by: Kolijn Wolfaardt <kolijn.wolfaardt@gmail.com>
Parts:
- SW0, SW1: footprint Buttons_Switches_SMD:SW_SPST_PTS645 -> RoBoC:SW_SPST_bigpads
Changed lines of the file:
@@
 F 0 "SW0" H 2150 6600 50  0000 C CNN
 F 1 "But 0" H 2150 6500 50  0000 C CNN
-F 2 "Buttons_Switches_SMD:SW_SPST_PTS645" H 1850 6550 60  0001 C CNN
+F 2 "RoBoC:SW_SPST_bigpads" H 1850 6550 60  0001 C CNN
 F 3 "" H 1850 6550 60  0000 C CNN
 	1    1850 6550
@@
 F 0 "SW1" H 3600 6600 50  0000 C CNN
 F 1 "But 1" H 3600 6500 50  0000 C CNN
-F 2 "Buttons_Switches_SMD:SW_SPST_PTS645" H 3300 6550 60  0001 C CNN
+F 2 "RoBoC:SW_SPST_bigpads" H 3300 6550 60  0001 C CNN
 F 3 "" H 3300 6550 60  0000 C CNN
 	1    3300 6550
