File: PCB Design/motors.sch (KiCad schematic (older format))
At the start: 17 parts, among them P3 Encoder 1, P4 Motor 1, P5 Motor 2, P6 Encoder 2, P7 PWM 1, P8 PWM 2, U2 LV8405V

Commit message: Did some fixes, added better footprint for the flyback diodes:
Re-routed camera bus so that there is more ground for the crystal.
Added ground pour keepouts under the MCU.
Changed the footprint for the motor flyback diodes.
Changed the camera module to have 24 pins, 2 won't be connected
Checked the footprints for dsPIC, MCP and LV8045
Increased thermal pad for voltage regulator

Signed-off-by: Kolijn Wolfaardt <kolijn.wolfaardt@gmail.com>
Parts:
- D10, D11, D12, D13, D14, D15, D16, D17: footprint Diodes_SMD:SOD-323 -> RoBoC:SOD-323
Changed lines of the file:
@@
 F 0 "D12" H 2800 4750 50  0000 C CNN
 F 1 "D" H 2800 4550 50  0000 C CNN
-F 2 "Diodes_SMD:SOD-323" H 2800 4650 60  0001 C CNN
+F 2 "RoBoC:SOD-323" H 2800 4650 60  0001 C CNN
 F 3 "" H 2800 4650 60  0000 C CNN
 	1    2800 4650
@@
 F 0 "D16" H 3100 4750 50  0000 C CNN
 F 1 "D" H 3100 4550 50  0000 C CNN
-F 2 "Diodes_SMD:SOD-323" H 3100 4650 60  0001 C CNN
+F 2 "RoBoC:SOD-323" H 3100 4650 60  0001 C CNN
 F 3 "" H 3100 4650 60  0000 C CNN
 	1    3100 4650
@@
 F 0 "D13" H 2800 5350 50  0000 C CNN
 F 1 "D" H 2800 5150 50  0000 C CNN
-F 2 "Diodes_SMD:SOD-323" H 2800 5250 60  0001 C CNN
+F 2 "RoBoC:SOD-323" H 2800 5250 60  0001 C CNN
 F 3 "" H 2800 5250 60  0000 C CNN
 	1    2800 5250
@@
 F 0 "D17" H 3100 5350 50  0000 C CNN
 F 1 "D" H 3100 5150 50  0000 C CNN
-F 2 "Diodes_SMD:SOD-323" H 3100 5250 60  0001 C CNN
+F 2 "RoBoC:SOD-323" H 3100 5250 60  0001 C CNN
 F 3 "" H 3100 5250 60  0000 C CNN
 	1    3100 5250
@@
 F 0 "D10" H 2750 3100 50  0000 C CNN
 F 1 "D" H 2750 2900 50  0000 C CNN
-F 2 "Diodes_SMD:SOD-323" H 2750 3000 60  0001 C CNN
+F 2 "RoBoC:SOD-323" H 2750 3000 60  0001 C CNN
 F 3 "" H 2750 3000 60  0000 C CNN
 	1    2750 3000
@@
 F 0 "D14" H 3050 3100 50  0000 C CNN
 F 1 "D" H 3050 2900 50  0000 C CNN
-F 2 "Diodes_SMD:SOD-323" H 3050 3000 60  0001 C CNN
+F 2 "RoBoC:SOD-323" H 3050 3000 60  0001 C CNN
 F 3 "" H 3050 3000 60  0000 C CNN
 	1    3050 3000
@@
 F 0 "D11" H 2750 3700 50  0000 C CNN
 F 1 "D" H 2750 3500 50  0000 C CNN
-F 2 "Diodes_SMD:SOD-323" H 2750 3600 60  0001 C CNN
+F 2 "RoBoC:SOD-323" H 2750 3600 60  0001 C CNN
 F 3 "" H 2750 3600 60  0000 C CNN
 	1    2750 3600
@@
 F 0 "D15" H 3050 3700 50  0000 C CNN
 F 1 "D" H 3050 3500 50  0000 C CNN
-F 2 "Diodes_SMD:SOD-323" H 3050 3600 60  0001 C CNN
+F 2 "RoBoC:SOD-323" H 3050 3600 60  0001 C CNN
 F 3 "" H 3050 3600 60  0000 C CNN
 	1    3050 3600

Commit message: Increased pad sizes for easy soldering, final commit before ordering
Signed-off-by: Kolijn Wolfaardt <kolijn.wolfaardt@gmail.com>
Parts:
- added C25, C26: 100nF, Capacitors_SMD:C_1206, symbol C
- U2: footprint Housings_SSOP:SSOP-16_4.4x5.2mm_Pitch0.65mm -> RoBoC:SSOP-16_4.4x5.2mm_Pitch0.65mm_Handsoldering
Connections:
- wire segments 70 -> 74
Changed lines of the file:
@@
 F 0 "U2" H 5600 3200 60  0000 C CNN
 F 1 "LV8405V" H 5600 4200 60  0000 C CNN
-F 2 "Housings_SSOP:SSOP-16_4.4x5.2mm_Pitch0.65mm" H 5800 3250 60  0001 C CNN
+F 2 "RoBoC:SSOP-16_4.4x5.2mm_Pitch0.65mm_Handsoldering" H 5800 3250 60  0001 C CNN
 F 3 "" H 5800 3250 60  0000 C CNN
 	1    5600 3700
@@
 Connection ~ 3100 4850
 Wire Wire Line
-	2700 4450 3100 4450
+	2700 4450 3400 4450
 Wire Wire Line
 	3100 4450 3100 4500
@@
 	2800 5400 2800 5450
 Wire Wire Line
-	2800 5450 3100 5450
+	2800 5450 3400 5450
 Wire Wire Line
 	2950 5450 2950 5500
@@
 Connection ~ 3050 3200
 Wire Wire Line
-	2650 2800 3050 2800
+	2650 2800 3350 2800
 Wire Wire Line
 	3050 2800 3050 2850
@@
 	2750 3750 2750 3800
 Wire Wire Line
-	2750 3800 3050 3800
+	2750 3800 3350 3800
 Wire Wire Line
 	2900 3800 2900 3850
@@
 	3050 3800 3050 3750
 Connection ~ 2900 3800
+$Comp
+L C C26
+U 1 1 5538C790
+P 3400 4950
+F 0 "C26" H 3425 5050 50  0000 L CNN
+F 1 "100nF" H 3425 4850 50  0000 L CNN
+F 2 "Capacitors_SMD:C_1206" H 3438 4800 30  0001 C CNN
+F 3 "" H 3400 4950 60  0000 C CNN
+	1    3400 4950
+	1    0    0    -1
+$EndComp
+$Comp
+L C C25
+U 1 1 5538C861
+P 3350 3300
+F 0 "C25" H 3375 3400 50  0000 L CNN
+F 1 "100nF" H 3375 3200 50  0000 L CNN
+F 2 "Capacitors_SMD:C_1206" H 3388 3150 30  0001 C CNN
+F 3 "" H 3350 3300 60  0000 C CNN
+	1    3350 3300
+	1    0    0    -1
+$EndComp
+Wire Wire Line
+	3350 2800 3350 3150
+Connection ~ 3050 2800
+Wire Wire Line
+	3350 3800 3350 3450
+Connection ~ 3050 3800
+Wire Wire Line
+	3400 4450 3400 4800
+Connection ~ 3100 4450
+Wire Wire Line
+	3400 5450 3400 5100
+Connection ~ 3100 5450
 $EndSCHEMATC
