File: PCB Design/usb.sch (KiCad schematic (older format))
At the start: 11 parts, among them CON1 USB-MICRO-B, U3 MCP2200, X1 12MHz

Commit message: Added initial footprint associations, caps and resistors.
Kicad is giving weird errors for the libraries and BOM generator.
The libraries have to be downloaded manually from github, and
then added.

Signed-off-by: Kolijn Wolfaardt <kolijn.wolfaardt@gmail.com>
Parts:
- C15, C16: value C -> 22pF; footprint (none) -> Capacitors_SMD:C_1206
- C17: footprint (none) -> Capacitors_SMD:C_1206
- CON1: footprint (none) -> USB
- D7, D8: footprint (none) -> LEDs:LED-1206
- R10, R11, R12: footprint (none) -> Resistors_SMD:R_1206
Changed lines of the file:
@@
 F 0 "U3" H 5550 2600 60  0000 C CNN
 F 1 "MCP2200" H 5550 3800 60  0000 C CNN
-F 2 "" H 5600 3200 60  0000 C CNN
+F 2 "" H 5600 3200 60  0001 C CNN
 F 3 "" H 5600 3200 60  0000 C CNN
 	1    5550 3200
@@
 F 0 "CON1" H 5500 5750 50  0000 C CNN
 F 1 "USB-MICRO-B" H 5650 5050 50  0000 C CNN
-F 2 "" H 5800 5300 50  0000 C CNN
+F 2 "USB" H 5800 5300 50  0001 C CNN
 F 3 "" H 5800 5300 50  0000 C CNN
 	1    5800 5400
@@
 F 0 "R11" V 9580 1700 50  0000 C CNN
 F 1 "220" V 9507 1701 50  0000 C CNN
-F 2 "" V 9430 1700 30  0000 C CNN
+F 2 "Resistors_SMD:R_1206" V 9430 1700 30  0001 C CNN
 F 3 "" H 9500 1700 30  0000 C CNN
 	1    9500 1700
@@
 F 0 "R12" V 9980 1700 50  0000 C CNN
 F 1 "220" V 9907 1701 50  0000 C CNN
-F 2 "" V 9830 1700 30  0000 C CNN
+F 2 "Resistors_SMD:R_1206" V 9830 1700 30  0001 C CNN
 F 3 "" H 9900 1700 30  0000 C CNN
 	1    9900 1700
@@
 F 0 "D7" H 9500 2350 50  0000 C CNN
 F 1 "LED" H 9500 2150 50  0000 C CNN
-F 2 "" H 9500 2250 60  0000 C CNN
+F 2 "LEDs:LED-1206" H 9500 2250 60  0001 C CNN
 F 3 "" H 9500 2250 60  0000 C CNN
 	1    9500 2250
@@
 F 0 "D8" H 9900 2350 50  0000 C CNN
 F 1 "LED" H 9900 2150 50  0000 C CNN
-F 2 "" H 9900 2250 60  0000 C CNN
+F 2 "LEDs:LED-1206" H 9900 2250 60  0001 C CNN
 F 3 "" H 9900 2250 60  0000 C CNN
 	1    9900 2250
@@
 F 0 "X1" H 2250 3350 50  0000 C CNN
 F 1 "12MHz" H 2250 3050 50  0000 C CNN
-F 2 "" H 2250 3200 60  0000 C CNN
+F 2 "" H 2250 3200 60  0001 C CNN
 F 3 "" H 2250 3200 60  0000 C CNN
 	1    2250 3200
@@
 P 1950 2800
 F 0 "C15" H 2000 2900 50  0000 L CNN
-F 1 "C" H 2000 2700 50  0000 L CNN
-F 2 "" H 1988 2650 30  0000 C CNN
+F 1 "22pF" H 2000 2700 50  0000 L CNN
+F 2 "Capacitors_SMD:C_1206" H 1988 2650 30  0001 C CNN
 F 3 "" H 1950 2800 60  0000 C CNN
 	1    1950 2800
@@
 P 1950 3600
 F 0 "C16" H 2000 3700 50  0000 L CNN
-F 1 "C" H 2000 3500 50  0000 L CNN
-F 2 "" H 1988 3450 30  0000 C CNN
+F 1 "22pF" H 2000 3500 50  0000 L CNN
+F 2 "Capacitors_SMD:C_1206" H 1988 3450 30  0001 C CNN
 F 3 "" H 1950 3600 60  0000 C CNN
 	1    1950 3600
@@
 F 0 "R10" V 6480 6050 50  0000 C CNN
 F 1 "18k" V 6407 6051 50  0000 C CNN
-F 2 "" V 6330 6050 30  0000 C CNN
+F 2 "Resistors_SMD:R_1206" V 6330 6050 30  0001 C CNN
 F 3 "" H 6400 6050 30  0000 C CNN
 	1    6400 6050
@@
 F 0 "C17" H 6750 6150 50  0000 L CNN
 F 1 "100nF" H 6750 5950 50  0000 L CNN
-F 2 "" H 6738 5900 30  0000 C CNN
+F 2 "Capacitors_SMD:C_1206" H 6738 5900 30  0001 C CNN
 F 3 "" H 6700 6050 60  0000 C CNN
 	1    6700 6050

Commit message: Added diodes to motor driver
Signed-off-by: Kolijn_Laptop <kolijn.wolfaardt@gmail.com>
Parts:
- CON1: footprint USB -> (none)
- U3: footprint (none) -> Housings_SOIC:SOIC-20_7.5x12.8mm_Pitch1.27mm
Changed lines of the file:
@@
 $EndDescr
 $Comp
-L +3V3 #PWR041
+L +3V3 #PWR044
 U 1 1 551026A6
 P 1800 1200
-F 0 "#PWR041" H 1800 1050 60  0001 C CNN
+F 0 "#PWR044" H 1800 1050 60  0001 C CNN
 F 1 "+3V3" H 1800 1340 60  0000 C CNN
 F 2 "" H 1800 1200 60  0000 C CNN
@@
 $EndComp
 $Comp
-L GND #PWR042
+L GND #PWR045
 U 1 1 551026AC
 P 1800 1350
-F 0 "#PWR042" H 1800 1100 60  0001 C CNN
+F 0 "#PWR045" H 1800 1100 60  0001 C CNN
 F 1 "GND" H 1800 1200 60  0000 C CNN
 F 2 "" H 1800 1350 60  0000 C CNN
@@
 F 0 "U3" H 5550 2600 60  0000 C CNN
 F 1 "MCP2200" H 5550 3800 60  0000 C CNN
-F 2 "" H 5600 3200 60  0001 C CNN
+F 2 "Housings_SOIC:SOIC-20_7.5x12.8mm_Pitch1.27mm" H 5600 3200 60  0001 C CNN
 F 3 "" H 5600 3200 60  0000 C CNN
 	1    5550 3200
@@
 MCU_RX
 $Comp
-L +3V3 #PWR043
+L +3V3 #PWR046
 U 1 1 55102790
 P 4200 2550
-F 0 "#PWR043" H 4200 2400 60  0001 C CNN
+F 0 "#PWR046" H 4200 2400 60  0001 C CNN
 F 1 "+3V3" H 4200 2690 60  0000 C CNN
 F 2 "" H 4200 2550 60  0000 C CNN
@@
 $EndComp
 $Comp
-L GND #PWR044
+L GND #PWR047
 U 1 1 551027AA
 P 6900 2850
-F 0 "#PWR044" H 6900 2600 60  0001 C CNN
+F 0 "#PWR047" H 6900 2600 60  0001 C CNN
 F 1 "GND" H 6900 2700 60  0000 C CNN
 F 2 "" H 6900 2850 60  0000 C CNN
@@
 F 0 "CON1" H 5500 5750 50  0000 C CNN
 F 1 "USB-MICRO-B" H 5650 5050 50  0000 C CNN
-F 2 "USB" H 5800 5300 50  0001 C CNN
+F 2 "" H 5800 5300 50  0001 C CNN
 F 3 "" H 5800 5300 50  0000 C CNN
 	1    5800 5400
@@
 	9900 1850 9900 2050
 $Comp
-L +3V3 #PWR045
+L +3V3 #PWR048
 U 1 1 55102C97
 P 9700 1350
-F 0 "#PWR045" H 9700 1200 60  0001 C CNN
+F 0 "#PWR048" H 9700 1200 60  0001 C CNN
 F 1 "+3V3" H 9700 1490 60  0000 C CNN
 F 2 "" H 9700 1350 60  0000 C CNN
@@
 $EndComp
 $Comp
-L GND #PWR046
+L GND #PWR049
 U 1 1 55102FBE
 P 1650 3700
-F 0 "#PWR046" H 1650 3450 60  0001 C CNN
+F 0 "#PWR049" H 1650 3450 60  0001 C CNN
 F 1 "GND" H 1650 3550 60  0000 C CNN
 F 2 "" H 1650 3700 60  0000 C CNN
@@
 USB_OSC2
 $Comp
-L GND #PWR047
+L GND #PWR050
 U 1 1 551032EF
 P 5200 5700
-F 0 "#PWR047" H 5200 5450 60  0001 C CNN
+F 0 "#PWR050" H 5200 5450 60  0001 C CNN
 F 1 "GND" H 5200 5550 60  0000 C CNN
 F 2 "" H 5200 5700 60  0000 C CNN
@@
 	5300 5200 4800 5200
 $Comp
-L GND #PWR048
+L GND #PWR051
 U 1 1 551035D3
 P 6400 6400
-F 0 "#PWR048" H 6400 6150 60  0001 C CNN
+F 0 "#PWR051" H 6400 6150 60  0001 C CNN
 F 1 "GND" H 6400 6250 60  0000 C CNN
 F 2 "" H 6400 6400 60  0000 C CNN
@@
 Connection ~ 6400 5300
 $Comp
-L +3V3 #PWR049
+L +3V3 #PWR052
 U 1 1 55103924
 P 7150 2950
-F 0 "#PWR049" H 7150 2800 60  0001 C CNN
+F 0 "#PWR052" H 7150 2800 60  0001 C CNN
 F 1 "+3V3" H 7150 3090 60  0000 C CNN
 F 2 "" H 7150 2950 60  0000 C CNN

Commit message: Added crystal footprint
Signed-off-by: Kolijn Wolfaardt <kolijn.wolfaardt@gmail.com>
Parts:
- removed X1: 12MHz, symbol CRYSTAL
- added X1: 12MHz, RoBoC:Crystal 6x 3.5 x 1.1mm, symbol CRYSTAL_SMD
Connections:
- wire segments 48 -> 49
Changed lines of the file:
@@
 $EndDescr
 $Comp
-L +3V3 #PWR044
+L +3V3 #PWR45
 U 1 1 551026A6
 P 1800 1200
-F 0 "#PWR044" H 1800 1050 60  0001 C CNN
+F 0 "#PWR45" H 1800 1050 60  0001 C CNN
 F 1 "+3V3" H 1800 1340 60  0000 C CNN
 F 2 "" H 1800 1200 60  0000 C CNN
@@
 $EndComp
 $Comp
-L GND #PWR045
+L GND #PWR46
 U 1 1 551026AC
 P 1800 1350
-F 0 "#PWR045" H 1800 1100 60  0001 C CNN
+F 0 "#PWR46" H 1800 1100 60  0001 C CNN
 F 1 "GND" H 1800 1200 60  0000 C CNN
 F 2 "" H 1800 1350 60  0000 C CNN
@@
 MCU_RX
 $Comp
-L +3V3 #PWR046
+L +3V3 #PWR47
 U 1 1 55102790
 P 4200 2550
-F 0 "#PWR046" H 4200 2400 60  0001 C CNN
+F 0 "#PWR47" H 4200 2400 60  0001 C CNN
 F 1 "+3V3" H 4200 2690 60  0000 C CNN
 F 2 "" H 4200 2550 60  0000 C CNN
@@
 $EndComp
 $Comp
-L GND #PWR047
+L GND #PWR50
 U 1 1 551027AA
 P 6900 2850
-F 0 "#PWR047" H 6900 2600 60  0001 C CNN
+F 0 "#PWR50" H 6900 2600 60  0001 C CNN
 F 1 "GND" H 6900 2700 60  0000 C CNN
 F 2 "" H 6900 2850 60  0000 C CNN
@@
 	9900 1850 9900 2050
 $Comp
-L +3V3 #PWR048
+L +3V3 #PWR52
 U 1 1 55102C97
 P 9700 1350
-F 0 "#PWR048" H 9700 1200 60  0001 C CNN
+F 0 "#PWR52" H 9700 1200 60  0001 C CNN
 F 1 "+3V3" H 9700 1490 60  0000 C CNN
 F 2 "" H 9700 1350 60  0000 C CNN
@@
 	9900 1350 9900 1550
 Connection ~ 9700 1350
-$Comp
-L CRYSTAL X1
-U 1 1 55102DA2
-P 2250 3200
-F 0 "X1" H 2250 3350 50  0000 C CNN
-F 1 "12MHz" H 2250 3050 50  0000 C CNN
-F 2 "" H 2250 3200 60  0001 C CNN
-F 3 "" H 2250 3200 60  0000 C CNN
-	1    2250 3200
-	0    1    1    0
-$EndComp
 $Comp
 L C C15
@@
 $EndComp
 $Comp
-L GND #PWR049
+L GND #PWR44
 U 1 1 55102FBE
 P 1650 3700
-F 0 "#PWR049" H 1650 3450 60  0001 C CNN
+F 0 "#PWR44" H 1650 3450 60  0001 C CNN
 F 1 "GND" H 1650 3550 60  0000 C CNN
 F 2 "" H 1650 3700 60  0000 C CNN
@@
 USB_OSC2
 $Comp
-L GND #PWR050
+L GND #PWR48
 U 1 1 551032EF
 P 5200 5700
-F 0 "#PWR050" H 5200 5450 60  0001 C CNN
+F 0 "#PWR48" H 5200 5450 60  0001 C CNN
 F 1 "GND" H 5200 5550 60  0000 C CNN
 F 2 "" H 5200 5700 60  0000 C CNN
@@
 	5300 5200 4800 5200
 $Comp
-L GND #PWR051
+L GND #PWR49
 U 1 1 551035D3
 P 6400 6400
-F 0 "#PWR051" H 6400 6150 60  0001 C CNN
+F 0 "#PWR49" H 6400 6150 60  0001 C CNN
 F 1 "GND" H 6400 6250 60  0000 C CNN
 F 2 "" H 6400 6400 60  0000 C CNN
@@
 Connection ~ 6400 5300
 $Comp
-L +3V3 #PWR052
+L +3V3 #PWR51
 U 1 1 55103924
 P 7150 2950
-F 0 "#PWR052" H 7150 2800 60  0001 C CNN
+F 0 "#PWR51" H 7150 2800 60  0001 C CNN
 F 1 "+3V3" H 7150 3090 60  0000 C CNN
 F 2 "" H 7150 2950 60  0000 C CNN
@@
 Connection ~ 6400 6300
 Wire Wire Line
-	2250 3600 2250 3500
+	2250 3400 2250 3600
 Connection ~ 2250 3600
 Wire Wire Line
-	2250 2900 2250 2800
+	2250 2800 2250 3000
 Connection ~ 2250 2800
 NoConn ~ 5300 5500
+$Comp
+L CRYSTAL_SMD X1
+U 1 1 55192ECE
+P 2250 3200
+F 0 "X1" H 2250 3290 50  0000 C CNN
+F 1 "12MHz" H 2280 3090 50  0000 L CNN
+F 2 "RoBoC:Crystal 6x 3.5 x 1.1mm" H 2250 3200 60  0001 C CNN
+F 3 "" H 2250 3200 60  0000 C CNN
+	1    2250 3200
+	0    1    1    0
+$EndComp
+Wire Wire Line
+	2150 3200 1650 3200
+Connection ~ 1650 3200
 $EndSCHEMATC

Commit message: Finished the footprint allocation, started on the PCB layout.-s
Parts:
- C15, C16: value 22pF -> 12pF
- CON1: value USB-MICRO-B -> USB; footprint (none) -> RoBoC:USB_Micro
- D7: value LED -> TX LED
- D8: value LED -> RX LED
Changed lines of the file:
@@
 $EndDescr
 $Comp
-L +3V3 #PWR45
+L +3V3 #PWR044
 U 1 1 551026A6
 P 1800 1200
-F 0 "#PWR45" H 1800 1050 60  0001 C CNN
+F 0 "#PWR044" H 1800 1050 60  0001 C CNN
 F 1 "+3V3" H 1800 1340 60  0000 C CNN
 F 2 "" H 1800 1200 60  0000 C CNN
@@
 $EndComp
 $Comp
-L GND #PWR46
+L GND #PWR045
 U 1 1 551026AC
 P 1800 1350
-F 0 "#PWR46" H 1800 1100 60  0001 C CNN
+F 0 "#PWR045" H 1800 1100 60  0001 C CNN
 F 1 "GND" H 1800 1200 60  0000 C CNN
 F 2 "" H 1800 1350 60  0000 C CNN
@@
 MCU_RX
 $Comp
-L +3V3 #PWR47
+L +3V3 #PWR046
 U 1 1 55102790
 P 4200 2550
-F 0 "#PWR47" H 4200 2400 60  0001 C CNN
+F 0 "#PWR046" H 4200 2400 60  0001 C CNN
 F 1 "+3V3" H 4200 2690 60  0000 C CNN
 F 2 "" H 4200 2550 60  0000 C CNN
@@
 $EndComp
 $Comp
-L GND #PWR50
+L GND #PWR047
 U 1 1 551027AA
 P 6900 2850
-F 0 "#PWR50" H 6900 2600 60  0001 C CNN
+F 0 "#PWR047" H 6900 2600 60  0001 C CNN
 F 1 "GND" H 6900 2700 60  0000 C CNN
 F 2 "" H 6900 2850 60  0000 C CNN
@@
 P 5800 5400
 F 0 "CON1" H 5500 5750 50  0000 C CNN
-F 1 "USB-MICRO-B" H 5650 5050 50  0000 C CNN
-F 2 "" H 5800 5300 50  0001 C CNN
+F 1 "USB" H 5650 5050 50  0000 C CNN
+F 2 "RoBoC:USB_Micro" H 5800 5300 50  0001 C CNN
 F 3 "" H 5800 5300 50  0000 C CNN
 	1    5800 5400
@@
 P 9500 2250
 F 0 "D7" H 9500 2350 50  0000 C CNN
-F 1 "LED" H 9500 2150 50  0000 C CNN
+F 1 "TX LED" H 9500 2150 50  0000 C CNN
 F 2 "LEDs:LED-1206" H 9500 2250 60  0001 C CNN
 F 3 "" H 9500 2250 60  0000 C CNN
@@
 P 9900 2250
 F 0 "D8" H 9900 2350 50  0000 C CNN
-F 1 "LED" H 9900 2150 50  0000 C CNN
+F 1 "RX LED" H 9900 2150 50  0000 C CNN
 F 2 "LEDs:LED-1206" H 9900 2250 60  0001 C CNN
 F 3 "" H 9900 2250 60  0000 C CNN
@@
 	9900 1850 9900 2050
 $Comp
-L +3V3 #PWR52
+L +3V3 #PWR048
 U 1 1 55102C97
 P 9700 1350
-F 0 "#PWR52" H 9700 1200 60  0001 C CNN
+F 0 "#PWR048" H 9700 1200 60  0001 C CNN
 F 1 "+3V3" H 9700 1490 60  0000 C CNN
 F 2 "" H 9700 1350 60  0000 C CNN
@@
 P 1950 2800
 F 0 "C15" H 2000 2900 50  0000 L CNN
-F 1 "22pF" H 2000 2700 50  0000 L CNN
+F 1 "12pF" H 2000 2700 50  0000 L CNN
 F 2 "Capacitors_SMD:C_1206" H 1988 2650 30  0001 C CNN
 F 3 "" H 1950 2800 60  0000 C CNN
@@
 P 1950 3600
 F 0 "C16" H 2000 3700 50  0000 L CNN
-F 1 "22pF" H 2000 3500 50  0000 L CNN
+F 1 "12pF" H 2000 3500 50  0000 L CNN
 F 2 "Capacitors_SMD:C_1206" H 1988 3450 30  0001 C CNN
 F 3 "" H 1950 3600 60  0000 C CNN
@@
 $EndComp
 $Comp
-L GND #PWR44
+L GND #PWR049
 U 1 1 55102FBE
 P 1650 3700
-F 0 "#PWR44" H 1650 3450 60  0001 C CNN
+F 0 "#PWR049" H 1650 3450 60  0001 C CNN
 F 1 "GND" H 1650 3550 60  0000 C CNN
 F 2 "" H 1650 3700 60  0000 C CNN
@@
 USB_OSC2
 $Comp
-L GND #PWR48
+L GND #PWR050
 U 1 1 551032EF
 P 5200 5700
-F 0 "#PWR48" H 5200 5450 60  0001 C CNN
+F 0 "#PWR050" H 5200 5450 60  0001 C CNN
 F 1 "GND" H 5200 5550 60  0000 C CNN
 F 2 "" H 5200 5700 60  0000 C CNN
@@
 	5300 5200 4800 5200
 $Comp
-L GND #PWR49
+L GND #PWR051
 U 1 1 551035D3
 P 6400 6400
-F 0 "#PWR49" H 6400 6150 60  0001 C CNN
+F 0 "#PWR051" H 6400 6150 60  0001 C CNN
 F 1 "GND" H 6400 6250 60  0000 C CNN
 F 2 "" H 6400 6400 60  0000 C CNN
@@
 Connection ~ 6400 5300
 $Comp
-L +3V3 #PWR51
+L +3V3 #PWR052
 U 1 1 55103924
 P 7150 2950
-F 0 "#PWR51" H 7150 2800 60  0001 C CNN
+F 0 "#PWR052" H 7150 2800 60  0001 C CNN
 F 1 "+3V3" H 7150 3090 60  0000 C CNN
 F 2 "" H 7150 2950 60  0000 C CNN
